File: Hardware/projecto ecu.kicad_pcb (KiCad board)
At the start: 2 copper layers, 60.5 x 43.5 mm, 14 parts, among them J2 Conn_01x04_Pin, J7 Screw_Terminal_01x02, J8 Screw_Terminal_01x02, SW1 SW_SPST

Commit message: Add files via upload
Parts:
- added G***: LOGO, LOGO, B.Cu at (159.5, 77.8)
- C6: footprint Capacitor_THT:C_Disc_D8.0mm_W5.0mm_P7.50mm -> Capacitor_THT:CP_Radial_D10.0mm_P3.50mm
- moved G*** 23.3 mm to (175.4, 62.0)
- moved C6 2.46 mm to (155.0, 61.8)
Routing:
- net VCC: track 46.4 -> 44.9 mm

Commit message: Add files via upload
Parts:
- moved G*** 2.64 mm to (159.6, 80.4)
- moved J7 1.67 mm to (139.3, 60.3)
- moved D2 0.22 mm to (192.2, 64.5)
Routing:
- net Net-(J7-Pin_2): track 8.05 -> 10.3 mm
- net VCC: track 44.9 -> 43.1 mm
- net Net-(D2-K): track 25.2 -> 25.8 mm
Changed lines of the file:
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@@
 		(pad "1" thru_hole circle
 			(at 0 0)
-			(size 1.4 1.4)
+			(size 2 2)
 			(drill 0.7)
 			(layers "*.Cu" "*.Mask")
@@
 			(pintype "passive")
 		)
-		(pad "2" thru_hole oval
+		(pad "2" thru_hole circle
 			(at 5.08 0)
-			(size 1.4 1.4)
+			(size 2 2)
 			(drill 0.7)
 			(layers "*.Cu" "*.Mask")
@@
 	(footprint "TerminalBlock_MetzConnect:TerminalBlock_MetzConnect_Type055_RT01502HDWU_1x02_P5.00mm_Horizontal"
 		(layer "F.Cu")
-		(at 141 60.25 -90)
+		(at 139.33 60.27 -90)
 		(descr "terminal block Metz Connect Type055_RT01502HDWU, 2 pins, pitch 5mm, size 10x8mm, drill diameter 1.3mm, pad diameter 2.5mm, https://www.metz-connect.com/externalfiles/310551/863212.PDF, script-generated using https://gitlab.com/kicad/libraries/kicad-footprint-generator/-/tree/master/scripts/TerminalBlock_MetzConnect")
 		(tags "THT terminal block Metz Connect Type055_RT01502HDWU pitch 5mm size 10x8mm drill 1.3mm pad 2.5mm")
@@
 	(footprint "Capacitor_THT:C_Axial_L3.8mm_D2.6mm_P7.50mm_Horizontal"
 		(layer "F.Cu")
-		(at 192.25 64.75 90)
+		(at 192.22 64.53 90)
 		(descr "C, Axial series, Axial, Horizontal, pin pitch=7.5mm, length*diameter=3.8*2.6mm^2, http://www.vishay.com/docs/45231/arseries.pdf")
 		(tags "C Axial series Axial Horizontal pin pitch 7.5mm  length 3.8mm diameter 2.6mm")
@@
 		(pad "1" thru_hole circle
 			(at 0 0 90)
-			(size 1.6 1.6)
+			(size 2 2)
 			(drill 0.8)
 			(layers "*.Cu" "*.Mask")
@@
 		(pad "2" thru_hole circle
 			(at 7.5 0 90)
-			(size 1.6 1.6)
+			(size 2 2)
 			(drill 0.8)
 			(layers "*.Cu" "*.Mask")
@@
 		(pad "1" thru_hole circle
 			(at 0 0)
-			(size 1.4 1.4)
+			(size 2 2)
 			(drill 0.7)
 			(layers "*.Cu" "*.Mask")
@@
 			(pintype "passive")
 		)
-		(pad "2" thru_hole oval
+		(pad "2" thru_hole circle
 			(at 5.08 0)
-			(size 1.4 1.4)
+			(size 2 2)
 			(drill 0.7)
 			(layers "*.Cu" "*.Mask")
@@
 			(at 1.75 6.25 0)
 			(layer "F.Fab")
+			(hide yes)
 			(effects
 				(font
@@
 		(model "C:/Users/Usuario/Desktop/Nueva carpeta (2)/LIBRERIA-KICAD/3D models/step down 360/MIni - 360.step"
 			(offset
-				(xyz 0 0 -16)
+				(xyz -0.5 -0.5 -16)
 			)
 			(scale
-				(xyz 1 1 1)
+				(xyz 0.9 1 1)
 			)
 			(rotate
@@
 			(layer "F.Fab")
 		)
-		(pad "1" thru_hole circle
-			(at -8.12 -9.9 270)
-			(size 2 2)
+		(pad "1" thru_hole oval
+			(at -8.12 -9.9)
+			(size 1.6 2)
 			(drill 1)
 			(layers "*.Cu" "*.Mask")
@@
 			(solder_mask_margin 0.102)
 		)
-		(pad "2" thru_hole circle
-			(at -8.12 -7.36 270)
-			(size 2 2)
+		(pad "2" thru_hole oval
+			(at -8.12 -7.36)
+			(size 1.6 2)
 			(drill 1)
 			(layers "*.Cu" "*.Mask")
@@
 			(solder_mask_margin 0.102)
 		)
-		(pad "3" thru_hole circle
-			(at -8.12 -4.82 270)
-			(size 2 2)
+		(pad "3" thru_hole oval
+			(at -8.12 -4.82)
+			(size 1.6 2)
 			(drill 1)
 			(layers "*.Cu" "*.Mask")
@@
 			(solder_mask_margin 0.102)
 		)
-		(pad "4" thru_hole circle
-			(at -8.12 -2.28 270)
-			(size 2 2)
+		(pad "4" thru_hole oval
+			(at -8.12 -2.28)
+			(size 1.6 2)
 			(drill 1)
 			(layers "*.Cu" "*.Mask")
@@
 			(solder_mask_margin 0.102)
 		)
-		(pad "5" thru_hole circle
-			(at -8.12 0.26 270)
-			(size 2 2)
+		(pad "5" thru_hole oval
+			(at -8.12 0.26)
+			(size 1.6 2)
 			(drill 1)
 			(layers "*.Cu" "*.Mask")
@@
 			(solder_mask_margin 0.102)
 		)
-		(pad "6" thru_hole circle
-			(at -8.12 2.8 270)
-			(size 2 2)
+		(pad "6" thru_hole oval
+			(at -8.12 2.8)
+			(size 1.6 2)
 			(drill 1)
 			(layers "*.Cu" "*.Mask")
@@
 			(solder_mask_margin 0.102)
 		)
-		(pad "7" thru_hole circle
-			(at -8.12 5.34 270)
-			(size 2 2)
+		(pad "7" thru_hole oval
+			(at -8.12 5.34)
+			(size 1.6 2)
 			(drill 1)
 			(layers "*.Cu" "*.Mask")
@@
 			(solder_mask_margin 0.102)
 		)
-		(pad "8" thru_hole circle
-			(at -8.12 7.88 270)
-			(size 2 2)
+		(pad "8" thru_hole oval
+			(at -8.12 7.88)
+			(size 1.6 2)
 			(drill 1)
 			(layers "*.Cu" "*.Mask")
@@
 			(solder_mask_margin 0.102)
 		)
-		(pad "9" thru_hole circle
-			(at 7.12 -9.9 270)
-			(size 2 2)
+		(pad "9" thru_hole oval
+			(at 7.12 -9.9)
+			(size 1.6 2)
 			(drill 1)
 			(layers "*.Cu" "*.Mask")
@@
 			(solder_mask_margin 0.102)
 		)
-		(pad "10" thru_hole circle
-			(at 7.12 -7.36 270)
-			(size 2 2)
+		(pad "10" thru_hole oval
+			(at 7.12 -7.36)
+			(size 1.6 2)
 			(drill 1)
 			(layers "*.Cu" "*.Mask")
@@
 			(solder_mask_margin 0.102)
 		)
-		(pad "11" thru_hole circle
-			(at 7.12 -4.82 270)
-			(size 2 2)
+		(pad "11" thru_hole oval
+			(at 7.12 -4.82)
+			(size 1.6 2)
 			(drill 1)
 			(layers "*.Cu" "*.Mask")
@@
 			(solder_mask_margin 0.102)
 		)
-		(pad "12" thru_hole circle
-			(at 7.12 -2.28 270)
-			(size 2 2)
+		(pad "12" thru_hole oval
+			(at 7.12 -2.28)
+			(size 1.6 2)
 			(drill 1)
 			(layers "*.Cu" "*.Mask")
@@
 			(solder_mask_margin 0.102)
 		)
-		(pad "13" thru_hole circle
-			(at 7.12 0.26 270)
-			(size 2 2)
+		(pad "13" thru_hole oval
+			(at 7.12 0.26)
+			(size 1.6 2)
 			(drill 1)
 			(layers "*.Cu" "*.Mask")
@@
 			(solder_mask_margin 0.102)
 		)
-		(pad "14" thru_hole circle
-			(at 7.12 2.8 270)
-			(size 2 2)
+		(pad "14" thru_hole oval
+			(at 7.12 2.8)
+			(size 1.6 2)
 			(drill 1)
 			(layers "*.Cu" "*.Mask")
@@
 			(solder_mask_margin 0.102)
 		)
-		(pad "15" thru_hole circle
-			(at 7.12 5.34 270)
-			(size 2 2)
+		(pad "15" thru_hole oval
+			(at 7.12 5.34)
+			(size 1.6 2)
 			(drill 1)
 			(layers "*.Cu" "*.Mask")
@@
 			(solder_mask_margin 0.102)
 		)
-		(pad "16" thru_hole circle
-			(at 7.12 7.88 270)
-			(size 2 2)
+		(pad "16" thru_hole oval
+			(at 7.12 7.88)
+			(size 1.6 2)
 			(drill 1)
 			(layers "*.Cu" "*.Mask")
@@
 			)
 			(scale
-				(xyz 1 1 1.1)
+				(xyz 1 1 1)
 			)
 			(rotate
@@
 	(footprint "LOGO"
 		(layer "B.Cu")
-		(at 159.5 77.8 180)
+		(at 159.61 80.44 180)
 		(property "Reference" "G***"
 			(at 0 0 0)
@@
 	)
 	(segment
-		(start 194.6 81.6)
+		(start 195.37 80.83)
 		(end 191.4 84.8)
 		(width 1)
@@
 	)
 	(segment
-		(start 192.25 64.75)
-		(end 192.25 66.65)
+		(start 192.22 64.78)
+		(end 192.22 66.62)
 		(width 1)
 		(layer "B.Cu")
@@
 	)
 	(segment
-		(start 194.6 69)
-		(end 194.6 81.6)
+		(start 191.4 84.8)
+		(end 191.4 87.62)
 		(width 1)
 		(layer "B.Cu")
@@
 	)
 	(segment
-		(start 191.4 84.8)
-		(end 191.4 87.62)
+		(start 192.22 66.62)
+		(end 195.37 69.77)
+		(width 1)
+		(layer "B.Cu")
+		(net 6)
+	)
+	(segment
+		(start 195.37 69.77)
+		(end 195.37 80.83)
 		(width 1)
 		(layer "B.Cu")
@@
 	)
 	(segment
-		(start 192.25 66.65)
-		(end 194.6 69)
+		(start 192.25 64.75)
+		(end 192.22 64.78)
 		(width 1)
 		(layer "B.Cu")
@@
 	)
 	(segment
+		(start 167.28 74.61)
+		(end 165.27 74.61)
+		(width 1)
+		(layer "B.Cu")
+		(net 7)
+	)
+	(segment
+		(start 165.27 74.61)
+		(end 155 64.34)
+		(width 1)
+		(layer "B.Cu")
+		(net 7)
+	)
+	(segment
 		(start 156.57 57.18)
 		(end 167.63 57.18)
@@
 	)
 	(segment
-		(start 157.13 69.53)
-		(end 155 67.4)
-		(width 1)
-		(layer "B.Cu")
-		(net 7)
-	)
-	(segment
-		(start 155 67.4)
+		(start 155 64.34)
 		(end 155 61.75)
 		(width 1)
@@
 	)
 	(segment
-		(start 167.28 74.61)
-		(end 165.61 74.61)
+		(start 153.15 61.75)
+		(end 155 61.75)
 		(width 1)
 		(layer "B.Cu")
@@
 	)
 	(segment
-		(start 160.53 69.53)
-		(end 157.13 69.53)
+		(start 141.55 65.27)
+		(end 141.57 65.25)
 		(width 1)
 		(layer "B.Cu")
-		(net 7)
+		(net 8)
 	)
 	(segment
-		(start 153.15 61.75)
-		(end 155 61.75)
+		(start 141.57 65.25)
+		(end 143.25 65.25)
 		(width 1)
 		(layer "B.Cu")
-		(net 7)
+		(net 8)
 	)
 	(segment
-		(start 165.61 74.61)
-		(end 160.53 69.53)
+		(start 141 65.25)
+		(end 141.57 65.25)
 		(width 1)
 		(layer "B.Cu")
-		(net 7)
+		(net 8)
 	)
 	(segment
-		(start 141 65.25)
-		(end 143.25 65.25)
+		(start 139.33 65.27)
+		(end 141.55 65.27)
 		(width 1)
 		(layer "B.Cu")
@@
 		(layer "B.Cu")
 		(hatch edge 0.5)
-		(connect_pads
-			(clearance 0.5)
+		(connect_pads yes
+			(clearance 1)
 		)
 		(min_thickness 0.25)
