File: Hardware/projecto ecu.kicad_sch (KiCad schematic)
At the start: 12 parts, among them J7 Screw_Terminal_01x02, J8 Screw_Terminal_01x02, SW1 SW_SPST

Commit message: Add files via upload
Parts:
- added J2: Conn_01x04_Pin, libreria rami:Mini360_step-down, symbol Connector:Conn_01x04_Pin
- C2: footprint Capacitor_THT:C_Axial_L3.8mm_D2.6mm_P7.50mm_Horizontal -> Capacitor_THT:C_Disc_D8.0mm_W5.0mm_P7.50mm
- C6: footprint Capacitor_THT:C_Axial_L3.8mm_D2.6mm_P7.50mm_Horizontal -> Capacitor_THT:CP_Radial_D10.0mm_P3.50mm
Connections:
- net GND: now also C6.2, J2.1 (Pin_1), J2.3 (Pin_3)
- net VCC: now also U2.4 (VCC), J2.2 (Pin_2); no longer D2.2 (A)
- new net 5V: D2.2 (A), J2.4 (Pin_4)
Other:
- note added: "ACTUADORES"
- note added: "BATERIA"
- note added: "CONTROLADOR DE LOS MOTORES"
- note added: "MICROCONTROLADOR"
- note added: "STEP DOWN 360 MINI"
- moved on the sheet: C6, D1, D2, R1
